Commit message: Adjust gripper joint upper limit value for 101.
Signed-off-by: Franco Cipollone <franco.c@ekumenlabs.com>

File: so_arm101_description/urdf/so_arm101_macro.xacro (robot description, xacro)
@@ -652,5 +652,5 @@
       <child link="${prefix}jaw_link" />
       <axis xyz="0 0 1" />
-      <limit effort="10" velocity="10" lower="0.0" upper="1." />
+      <limit effort="10" velocity="10" lower="0.0" upper="1.70" />
     </joint>
     <transmission name="${prefix}gripper_trans">
